File: schematic/schematic.kicad_sch (KiCad schematic)
At the start: 7 parts, among them K1 TIANBO-HJR-4102-L, U1 Pico

Commit message: wip
Parts:
- added SW1: SW_DPDT_x2, symbol Switch:SW_DPDT_x2
- added U2: L7805, symbol Regulator_Linear:L7805
Connections:
- net +10V: now also SW1.2 (B), U2.1 (IN); no longer K1.12, U1.39 (VSYS)
- net GND: now also U1.3 (GND), U2.2 (GND); no longer K1.8, U1.23 (GND)
- net at D3.1 (K): now also R2.2, U1.33 (AGND); no longer U1.5 (GPIO3)
- net at K1.5: now also U1.23 (GND); no longer U1.24 (GPIO18)
- net at R1.2: now also D2.1 (A), U1.29 (GPIO22); no longer U1.4 (GPIO2)
- net at U1.21 (GPIO16): now also K1.8
- net at U1.31 (GPIO26_ADC0): now also D2.2 (K), R2.1
- net at U1.6 (GPIO4): no longer R2.1
- net at U1.7 (GPIO5): no longer D2.2 (K)
- new net: K1.12, SW1.1 (A)
- new net 5V: U1.39 (VSYS), U2.3 (OUT)
Other:
- moved on the sheet: D2, D3, High-Voltage-LED1, K1, R1, R2, U1

Commit message: wip
Parts:
- renumbered High-Voltage-LED1 to 12V-LED1
Connections:
- net +10V renamed +12V
Changed lines of the file:
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@@
-    )
-  )
-  (symbol (lib_id "power:+10V") (at 46.99 24.13 90) (unit 1)
-    (in_bom yes) (on_board yes) (dnp no)
-    (property "Reference" "#PWR01" (at 50.8 24.13 0)
-      (effects (font (size 1.27 1.27)) hide)
-    )
-    (property "Value" "+10V" (at 41.91 21.59 90)
-      (effects (font (size 1.27 1.27)) (justify right))
-    )
-    (property "Footprint" "" (at 46.99 24.13 0)
-      (effects (font (size 1.27 1.27)) hide)
-    )
-    (property "Datasheet" "" (at 46.99 24.13 0)
-      (effects (font (size 1.27 1.27)) hide)
-    )
-    (pin "1")
-    (instances
-      (project "schematic"
-        (path "/46000928-40e7-4132-8b6b-3b3af6202dd3"
-          (reference "#PWR01") (unit 1)
-        )
-      )
     )
   )
@@
   (symbol (lib_id "Device:LED") (at 130.81 86.36 270) (unit 1)
     (in_bom yes) (on_board yes) (dnp no)
-    (property "Reference" "High-Voltage-LED1" (at 143.51 85.09 90)
-      (effects (font (size 1.27 1.27)))
-    )
-    (property "Value" "LED" (at 143.51 87.63 90)
+    (property "Reference" "12V-LED1" (at 139.7 85.09 90)
+      (effects (font (size 1.27 1.27)))
+    )
+    (property "Value" "LED" (at 139.7 87.63 90)
       (effects (font (size 1.27 1.27)))
     )
@@
       (project "schematic"
         (path "/46000928-40e7-4132-8b6b-3b3af6202dd3"
-          (reference "High-Voltage-LED1") (unit 1)
-        )
-      )
-    )
-  )
-  (symbol (lib_id "power:+10V") (at 127 129.54 90) (unit 1)
-    (in_bom yes) (on_board yes) (dnp no)
-    (property "Reference" "#PWR03" (at 130.81 129.54 0)
-      (effects (font (size 1.27 1.27)) hide)
-    )
-    (property "Value" "+10V" (at 124.46 132.08 90)
-      (effects (font (size 1.27 1.27)) (justify right))
-    )
-    (property "Footprint" "" (at 127 129.54 0)
-      (effects (font (size 1.27 1.27)) hide)
-    )
-    (property "Datasheet" "" (at 127 129.54 0)
-      (effects (font (size 1.27 1.27)) hide)
-    )
-    (pin "1")
-    (instances
-      (project "schematic"
-        (path "/46000928-40e7-4132-8b6b-3b3af6202dd3"
-          (reference "#PWR03") (unit 1)
+          (reference "12V-LED1") (unit 1)
+        )
+      )
+    )
+  )
+  (symbol (lib_id "power:+12V") (at 46.99 24.13 90) (unit 1)
+    (in_bom yes) (on_board yes) (dnp no) (fields_autoplaced)
+    (property "Reference" "#PWR06" (at 50.8 24.13 0)
+      (effects (font (size 1.27 1.27)) hide)
+    )
+    (property "Value" "+12V" (at 43.18 24.13 90)
+      (effects (font (size 1.27 1.27)) (justify left))
+    )
+    (property "Footprint" "" (at 46.99 24.13 0)
+      (effects (font (size 1.27 1.27)) hide)
+    )
+    (property "Datasheet" "" (at 46.99 24.13 0)
+      (effects (font (size 1.27 1.27)) hide)
+    )
+    (pin "1")
+    (instances
+      (project "schematic"
+        (path "/46000928-40e7-4132-8b6b-3b3af6202dd3"
+          (reference "#PWR06") (unit 1)
         )
       )
@@
         )
       )
+    )
+  )
+  (symbol (lib_id "power:+12V") (at 127 129.54 90) (unit 1)
+    (in_bom yes) (on_board yes) (dnp no) (fields_autoplaced)
+    (property "Reference" "#PWR01" (at 130.81 129.54 0)
+      (effects (font (size 1.27 1.27)) hide)
+    )
+    (property "Value" "+12V" (at 123.19 129.54 90)
+      (effects (font (size 1.27 1.27)) (justify left))
+    )
+    (property "Footprint" "" (at 127 129.54 0)
+      (effects (font (size 1.27 1.27)) hide)
+    )
+    (property "Datasheet" "" (at 127 129.54 0)
+      (effects (font (size 1.27 1.27)) hide)
+    )
+    (pin "1")
+    (instances
+      (project "schematic"
+        (path "/46000928-40e7-4132-8b6b-3b3af6202dd3"
+          (reference "#PWR01") (unit 1)
+        )
+      )
